File: Main PCB/Rob_Dev_Board.kicad_pcb (KiCad board)
At the start: 4 copper layers, 90 x 76 mm, 21 parts, among them J1 TYPE-C-31-M-12, J10 XT60PW-M, J11 XT60PW-M, J12 XT60PW-M, J2 XT60PW-M, J3 XT60PW-M, J4 XT60PW-M, J5 XT60PW-M, J6 XT60PW-M, J7 XT60PW-M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

Commit message: jawndice
Parts:
- moved J3 25.6 mm to (85.0, 63.0)
- moved J2 0.75 mm to (143.2, 79.0)
Changed lines of the file:
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@@
 	(footprint "XT60PW-M Connector:AMASS_XT60PW-M"
 		(layer "F.Cu")
-		(at 105 79)
+		(at 85 63)
 		(property "Reference" "J3"
 			(at -4.8236 -13.51498 0)
@@
 	(footprint "XT60PW-M Connector:AMASS_XT60PW-M"
 		(layer "F.Cu")
-		(at 142.5 79)
+		(at 143.25 79)
 		(property "Reference" "J2"
 			(at -4.8236 -13.51498 0)
