File: Main PCB/Rob_Dev_Board.kicad_pcb (KiCad board)
At the start: 4 copper layers, 90 x 76 mm, 21 parts, among them J1 TYPE-C-31-M-12, J10 XT60PW-M, J11 XT60PW-M, J12 XT60PW-M, J2 XT60PW-M, J3 XT60PW-M, J4 XT60PW-M, J5 XT60PW-M, J6 XT60PW-M, J7 XT60PW-M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

Commit message: more testing
Parts:
- moved J11 3.78 mm to (197.5, 67.0)
Changed lines of the file:
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@@
 	(footprint "XT60PW-M Connector:AMASS_XT60PW-M"
 		(layer "F.Cu")
-		(at 193.75 67.5)
+		(at 197.5 67)
 		(property "Reference" "J11"
 			(at -4.8236 -13.51498 0)

Commit message: testing more
Parts:
- moved J2 18.0 mm to (144.0, 61.0)
Changed lines of the file:
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@@
 	(footprint "XT60PW-M Connector:AMASS_XT60PW-M"
 		(layer "F.Cu")
-		(at 143.25 79)
+		(at 144 61)
 		(property "Reference" "J2"
 			(at -4.8236 -13.51498 0)
