File: hardware/Robodev/esp32.kicad_sch (KiCad schematic)
At the start: 31 parts, among them X1 USB4085-GF-A

Commit message: Add Board field to all schematic symbols for KiKit split
Assigns a hidden 'Board' property to every component across all 8
schematic sheets (263 symbols total) to support splitting the design
into two KiCad PCBs using `kikit separate`:

- Board="power"  — XT60 input, reverse-protection, XL4016 regulators
  (VMOT/VSTEP/VSERVO), LM2596 5V, AP2112K 3.3V, DRV8874 DC motor
  drivers ×4, TMC2209 stepper drivers ×2, PCA9685 servo controller,
  and all associated passives and motor/servo output connectors.

- Board="main"   — STM32G431 MCU, ESP32-C3 WiFi module, SN65HVD230
  CAN transceiver, 74HC595 SPI shift registers, BMI270 IMU, ADS1115
  ADC, PCF8574 GPIO expander, TCA9548A I2C muxes, USB connector, and
  all associated headers and passives.

The field is hidden in the schematic editor (hide=yes). Once the
inter-board connector pair is added, run:

  kikit separate --source 'field; field: Board; value: power' \
    Robodev.kicad_pcb power_board.kicad_pcb
  kikit separate --source 'field; field: Board; value: main' \
    Robodev.kicad_pcb main_board.kicad_pcb

Co-Authored-By: Claude Sonnet 4.6 <noreply@anthropic.com>
Parts:
- C_CAN1, C_NRST1, C_VBAT1, C_VDD1, C_VDD2, C_VDD3, C_VDD4, C_VDDA1, C_VDDA2, C_VDDBULK1, C_VREF1, C_VREF2, J_ADC1, J_ADC2, J_ADC3, J_CAN1, J_ENC1, J_ENC2, J_GPIO1, J_SWD1, J_UART2, J_UART_DBG1, R_BOOT0, R_CAN_TERM1, R_S1EN1, R_S2EN1, SW_BOOT1, SW_RESET1, U_CAN1, U_MCU1, X1: Board (none) -> main
