File: hardware/Robodev/i2c_bus.kicad_sch (KiCad schematic)
At the start: 34 parts

Commit message: Add Board field to all schematic symbols for KiKit split
Assigns a hidden 'Board' property to every component across all 8
schematic sheets (263 symbols total) to support splitting the design
into two KiCad PCBs using `kikit separate`:

- Board="power"  — XT60 input, reverse-protection, XL4016 regulators
  (VMOT/VSTEP/VSERVO), LM2596 5V, AP2112K 3.3V, DRV8874 DC motor
  drivers ×4, TMC2209 stepper drivers ×2, PCA9685 servo controller,
  and all associated passives and motor/servo output connectors.

- Board="main"   — STM32G431 MCU, ESP32-C3 WiFi module, SN65HVD230
  CAN transceiver, 74HC595 SPI shift registers, BMI270 IMU, ADS1115
  ADC, PCF8574 GPIO expander, TCA9548A I2C muxes, USB connector, and
  all associated headers and passives.

The field is hidden in the schematic editor (hide=yes). Once the
inter-board connector pair is added, run:

  kikit separate --source 'field; field: Board; value: power' \
    Robodev.kicad_pcb power_board.kicad_pcb
  kikit separate --source 'field; field: Board; value: main' \
    Robodev.kicad_pcb main_board.kicad_pcb

Co-Authored-By: Claude Sonnet 4.6 <noreply@anthropic.com>
Parts:
- C_ADC1, C_GPIO1, C_MUX1, C_MUX2, J_GPIO_EXP1, J_GPIO_GND1, J_GPIO_PWR1, J_MUX1_CH0, J_MUX1_CH1, J_MUX1_CH2, J_MUX1_CH3, J_MUX1_CH4, J_MUX1_CH5, J_MUX1_CH6, J_MUX1_CH7, J_MUX2_CH0, J_MUX2_CH1, J_MUX2_CH2, J_MUX2_CH3, J_MUX2_CH4, J_MUX2_CH5, J_MUX2_CH6, J_MUX2_CH7, J_OLED1, R_GPIO_A0, R_GPIO_A1, R_GPIO_A2, R_GPIO_INT1, R_MUX1_RST1, R_MUX2_RST1, U_ADC1, U_GPIO1, U_MUX1, U_MUX2: Board (none) -> main
