File: hardware/Robodev/motor_dc.kicad_sch (KiCad schematic)
At the start: 48 parts

Commit message: Add Board field to all schematic symbols for KiKit split
Assigns a hidden 'Board' property to every component across all 8
schematic sheets (263 symbols total) to support splitting the design
into two KiCad PCBs using `kikit separate`:

- Board="power"  — XT60 input, reverse-protection, XL4016 regulators
  (VMOT/VSTEP/VSERVO), LM2596 5V, AP2112K 3.3V, DRV8874 DC motor
  drivers ×4, TMC2209 stepper drivers ×2, PCA9685 servo controller,
  and all associated passives and motor/servo output connectors.

- Board="main"   — STM32G431 MCU, ESP32-C3 WiFi module, SN65HVD230
  CAN transceiver, 74HC595 SPI shift registers, BMI270 IMU, ADS1115
  ADC, PCF8574 GPIO expander, TCA9548A I2C muxes, USB connector, and
  all associated headers and passives.

The field is hidden in the schematic editor (hide=yes). Once the
inter-board connector pair is added, run:

  kikit separate --source 'field; field: Board; value: power' \
    Robodev.kicad_pcb power_board.kicad_pcb
  kikit separate --source 'field; field: Board; value: main' \
    Robodev.kicad_pcb main_board.kicad_pcb

Co-Authored-By: Claude Sonnet 4.6 <noreply@anthropic.com>
Parts:
- C_CP1, C_CP2, C_CP3, C_CP4, C_VCP1, C_VCP2, C_VCP3, C_VCP4, C_VM1, C_VM1_DEC1, C_VM2, C_VM2_DEC2, C_VM3, C_VM3_DEC3, C_VM4, C_VM4_DEC4, J_M1, J_M2, J_M3, J_M4, LED_FAULT1, LED_FAULT2, LED_FAULT3, LED_FAULT4, R_FAULT_LED1, R_FAULT_LED2, R_FAULT_LED3, R_FAULT_LED4, R_FAULT_PU1, R_FAULT_PU2, R_FAULT_PU3, R_FAULT_PU4, R_IMODE1, R_IMODE2, R_IMODE3, R_IMODE4, R_IPROPI1, R_IPROPI2, R_IPROPI3, R_IPROPI4, R_NSLEEP1, R_NSLEEP2, R_NSLEEP3, R_NSLEEP4, U_M1, U_M2, U_M3, U_M4: Board (none) -> power
