File: hardware/Robodev/motor_servo.kicad_sch (KiCad schematic)
At the start: 30 parts

Commit message: Add Board field to all schematic symbols for KiKit split
Assigns a hidden 'Board' property to every component across all 8
schematic sheets (263 symbols total) to support splitting the design
into two KiCad PCBs using `kikit separate`:

- Board="power"  — XT60 input, reverse-protection, XL4016 regulators
  (VMOT/VSTEP/VSERVO), LM2596 5V, AP2112K 3.3V, DRV8874 DC motor
  drivers ×4, TMC2209 stepper drivers ×2, PCA9685 servo controller,
  and all associated passives and motor/servo output connectors.

- Board="main"   — STM32G431 MCU, ESP32-C3 WiFi module, SN65HVD230
  CAN transceiver, 74HC595 SPI shift registers, BMI270 IMU, ADS1115
  ADC, PCF8574 GPIO expander, TCA9548A I2C muxes, USB connector, and
  all associated headers and passives.

The field is hidden in the schematic editor (hide=yes). Once the
inter-board connector pair is added, run:

  kikit separate --source 'field; field: Board; value: power' \
    Robodev.kicad_pcb power_board.kicad_pcb
  kikit separate --source 'field; field: Board; value: main' \
    Robodev.kicad_pcb main_board.kicad_pcb

Co-Authored-By: Claude Sonnet 4.6 <noreply@anthropic.com>
Parts:
- C_VDD_BULK_SERVO1, C_VDD_SERVO1, C_VSERVO_BULK1, C_VSERVO_DEC1, J_SV0, J_SV1, J_SV10, J_SV11, J_SV12, J_SV13, J_SV14, J_SV15, J_SV2, J_SV3, J_SV4, J_SV5, J_SV6, J_SV7, J_SV8, J_SV9, R_A0, R_A1, R_A2, R_A3, R_A4, R_A5, R_OE1, R_SCL1, R_SDA1, U_SERVO1: Board (none) -> power
