File: hardware/Robodev/motor_stepper.kicad_sch (KiCad schematic)
At the start: 35 parts

Commit message: Add Board field to all schematic symbols for KiKit split
Assigns a hidden 'Board' property to every component across all 8
schematic sheets (263 symbols total) to support splitting the design
into two KiCad PCBs using `kikit separate`:

- Board="power"  — XT60 input, reverse-protection, XL4016 regulators
  (VMOT/VSTEP/VSERVO), LM2596 5V, AP2112K 3.3V, DRV8874 DC motor
  drivers ×4, TMC2209 stepper drivers ×2, PCA9685 servo controller,
  and all associated passives and motor/servo output connectors.

- Board="main"   — STM32G431 MCU, ESP32-C3 WiFi module, SN65HVD230
  CAN transceiver, 74HC595 SPI shift registers, BMI270 IMU, ADS1115
  ADC, PCF8574 GPIO expander, TCA9548A I2C muxes, USB connector, and
  all associated headers and passives.

The field is hidden in the schematic editor (hide=yes). Once the
inter-board connector pair is added, run:

  kikit separate --source 'field; field: Board; value: power' \
    Robodev.kicad_pcb power_board.kicad_pcb
  kikit separate --source 'field; field: Board; value: main' \
    Robodev.kicad_pcb main_board.kicad_pcb

Co-Authored-By: Claude Sonnet 4.6 <noreply@anthropic.com>
Parts:
- C_5VOUT1, C_5VOUT2, C_CPS1, C_CPS2, C_VCC1, C_VCC2, C_VCPS1, C_VCPS2, C_VREFS1, C_VREFS2, C_VS1, C_VS1_DEC1, C_VS2, C_VS2_DEC2, J_S1, J_S1_DIAG1, J_S2, J_S2_DIAG1, R_CLK1, R_CLK2, R_MS1_S2, R_SENSE_SA1, R_SENSE_SA2, R_SENSE_SB1, R_SENSE_SB2, R_SPREAD1, R_SPREAD2, R_UART_S1, R_UART_S2, R_VREF_H1, R_VREF_H2, R_VREF_L1, R_VREF_L2, U_S1, U_S2: Board (none) -> power
