File: hardware/Robodev/power.kicad_sch (KiCad schematic)
At the start: 45 parts

Commit message: Add Board field to all schematic symbols for KiKit split
Assigns a hidden 'Board' property to every component across all 8
schematic sheets (263 symbols total) to support splitting the design
into two KiCad PCBs using `kikit separate`:

- Board="power"  — XT60 input, reverse-protection, XL4016 regulators
  (VMOT/VSTEP/VSERVO), LM2596 5V, AP2112K 3.3V, DRV8874 DC motor
  drivers ×4, TMC2209 stepper drivers ×2, PCA9685 servo controller,
  and all associated passives and motor/servo output connectors.

- Board="main"   — STM32G431 MCU, ESP32-C3 WiFi module, SN65HVD230
  CAN transceiver, 74HC595 SPI shift registers, BMI270 IMU, ADS1115
  ADC, PCF8574 GPIO expander, TCA9548A I2C muxes, USB connector, and
  all associated headers and passives.

The field is hidden in the schematic editor (hide=yes). Once the
inter-board connector pair is added, run:

  kikit separate --source 'field; field: Board; value: power' \
    Robodev.kicad_pcb power_board.kicad_pcb
  kikit separate --source 'field; field: Board; value: main' \
    Robodev.kicad_pcb main_board.kicad_pcb

Co-Authored-By: Claude Sonnet 4.6 <noreply@anthropic.com>
Parts:
- CC_IN_3V3, C_FB_VMOT1, C_FB_VSERVO1, C_FB_VSTEP1, C_IN_5V1, C_IN_VMOT1, C_IN_VSERVO1, C_IN_VSTEP1, C_OUT_3V3, C_OUT_5V1, C_OUT_VMOT1, C_OUT_VSERVO1, C_OUT_VSTEP1, C_VC_MOT1, C_VC_SERVO1, C_VC_STEP1, D_CATCH1, D_MOT1, D_SERVO1, D_STEP1, J_BENCH1, J_XT60, L_5V1, L_VMOT1, L_VSERVO1, L_VSTEP1, NT1, Q_REVPROT1, RV_VMOT1, RV_VSERVO1, RV_VSTEP1, R_FB_VMOT1, R_FB_VSERVO1, R_FB_VSTEP1, R_GATE_BLD1, R_GATE_PD1, R_MON_VIN_H1, R_MON_VIN_L1, SW_MAIN1, U_3V3, U_5V1, U_VMOT1, U_VSERVO1, U_VSTEP1: Board (none) -> power
- D_USB1: Board (none) -> main
