File: hardware/Robodev/spi_bus.kicad_sch (KiCad schematic)
At the start: 31 parts

Commit message: Add Board field to all schematic symbols for KiKit split
Assigns a hidden 'Board' property to every component across all 8
schematic sheets (263 symbols total) to support splitting the design
into two KiCad PCBs using `kikit separate`:

- Board="power"  — XT60 input, reverse-protection, XL4016 regulators
  (VMOT/VSTEP/VSERVO), LM2596 5V, AP2112K 3.3V, DRV8874 DC motor
  drivers ×4, TMC2209 stepper drivers ×2, PCA9685 servo controller,
  and all associated passives and motor/servo output connectors.

- Board="main"   — STM32G431 MCU, ESP32-C3 WiFi module, SN65HVD230
  CAN transceiver, 74HC595 SPI shift registers, BMI270 IMU, ADS1115
  ADC, PCF8574 GPIO expander, TCA9548A I2C muxes, USB connector, and
  all associated headers and passives.

The field is hidden in the schematic editor (hide=yes). Once the
inter-board connector pair is added, run:

  kikit separate --source 'field; field: Board; value: power' \
    Robodev.kicad_pcb power_board.kicad_pcb
  kikit separate --source 'field; field: Board; value: main' \
    Robodev.kicad_pcb main_board.kicad_pcb

Co-Authored-By: Claude Sonnet 4.6 <noreply@anthropic.com>
Parts:
- C_595A1, C_595B1, C_IMU_VDD1, C_IMU_VDDIO1, C_WIFI_1, C_WIFI_2, J_SPI1, J_SPI10, J_SPI11, J_SPI12, J_SPI13, J_SPI14, J_SPI15, J_SPI2, J_SPI3, J_SPI4, J_SPI5, J_SPI6, J_SPI7, J_SPI8, J_SPI9, J_WIFI_UART1, R_595A_SCLR1, R_595B_SCLR1, R_IO2_PULLUP_STRAP1, R_WIFI_EN1, R_WIFI_IO0, U_595A1, U_595B1, U_IMU1, U_WIFI1: Board (none) -> main
